File: oscilador_rampa.sch (KiCad schematic (older format))
At the start: 15 parts, among them IC1 4011, P10 4k7, T1 2N3904, T2 Q_NJFET_DGS, T3 Q_NJFET_DGS

Commit message: añado el conversor exponencial y mezclador
Parts:
- gave numbers to parts that had none: 2
Connections:
- net at IC1.2, P10.1, R18.2: now also D1.2 (A), D2.1 (K)
- net currexp renamed exp
Changed lines of the file:
@@
 $Descr A4 11693 8268
 encoding utf-8
-Sheet 2 2
+Sheet 2 4
 Title "Voltage Controlled Oscillator"
 Date ""
@@
 $EndComp
 $Comp
-L R R?
+L R R18
 U 1 1 59D4F972
 P 5400 3650
-F 0 "R?" V 5480 3650 50  0000 C CNN
+F 0 "R18" V 5480 3650 50  0000 C CNN
 F 1 "R" V 5400 3650 50  0000 C CNN
 F 2 "" V 5330 3650 50  0001 C CNN
@@
 $EndComp
 $Comp
-L POT P?
+L POT P9
 U 1 1 59D4F9A3
 P 3150 2850
-F 0 "P?" V 2975 2850 50  0000 C CNN
+F 0 "P9" V 2975 2850 50  0000 C CNN
 F 1 "2k2" V 3050 2850 50  0000 C CNN
 F 2 "" H 3150 2850 50  0001 C CNN
@@
 $EndComp
 Text HLabel 2800 3700 0    60   Input ~ 0
-currexp
+exp
 Text HLabel 2800 3950 0    60   Input ~ 0
 GND
@@
 -15V
 Wire Wire Line
-	4200 3550 4200 3650
-Wire Wire Line
-	4200 3650 4200 4450
-Wire Wire Line
-	4200 3650 4550 3650
-Wire Wire Line
-	4550 3650 5250 3650
+	4200 3550 4200 4450
+Wire Wire Line
+	4200 3650 5250 3650
 Wire Wire Line
 	4550 3650 4550 3750
@@
 	4550 4150 4700 4150
 Wire Wire Line
-	5000 4350 5000 4400
-Wire Wire Line
-	5000 4400 5000 4450
-Wire Wire Line
-	5000 4750 5000 4800
-Wire Wire Line
-	5000 4800 5000 5000
-Wire Wire Line
-	5550 3650 6000 3650
-Wire Wire Line
-	6000 3650 6050 3650
+	5000 4350 5000 4450
+Wire Wire Line
+	5000 4750 5000 5000
+Wire Wire Line
+	5550 3650 6050 3650
 Wire Wire Line
 	6050 3450 6050 2800
 Wire Wire Line
-	6050 1650 6050 2000
-Wire Wire Line
-	6050 2000 6050 2500
+	6050 1650 6050 2500
 Wire Wire Line
 	5750 2000 5750 2900
-Wire Wire Line
-	5750 3200 5750 3800
 Wire Wire Line
 	6000 3950 6000 3650
@@
 	5000 2950 5000 3950
 Wire Wire Line
-	4200 2950 4600 2950
-Wire Wire Line
-	4600 2950 5000 2950
+	4200 2950 5000 2950
 Wire Wire Line
 	4200 2950 4200 3150
@@
 Connection ~ 5000 4400
 Wire Wire Line
-	5750 4250 6000 4250
-Wire Wire Line
-	6000 4250 6150 4250
+	5750 4250 6150 4250
 Wire Wire Line
 	6150 4250 6150 4100
@@
 Connection ~ 6000 4250
 Wire Wire Line
-	3150 2500 3150 2600
-Wire Wire Line
-	3150 2600 3150 2700
-Wire Wire Line
-	3150 2600 3350 2600
-Wire Wire Line
-	3350 2600 3500 2600
+	3150 2500 3150 2700
+Wire Wire Line
+	3150 2600 3500 2600
 Connection ~ 3150 2600
 Wire Wire Line
@@
 	3150 2200 3150 2000
 Wire Wire Line
-	3150 2000 3450 2000
-Wire Wire Line
-	3450 2000 5750 2000
-Wire Wire Line
-	5750 2000 6050 2000
+	3150 2000 6050 2000
 Connection ~ 6050 2000
 Wire Wire Line
@@
 	7400 2400 4150 2400
 Wire Wire Line
-	3150 3000 3150 3350
-Wire Wire Line
-	3150 3350 3150 3700
+	3150 3000 3150 3700
 Wire Wire Line
 	3150 3700 2800 3700
@@
 Connection ~ 3150 3350
 Connection ~ 5750 2000
+Wire Wire Line
+	5750 3200 5750 3800
+Connection ~ 5750 3650
 $EndSCHEMATC
