File: ramp2triangle.sch (KiCad schematic (older format))
At the start: 0 parts

Commit message: sawtooh 2 triangle
Parts:
- added C13: 1n, symbol C
- added C8: 680, symbol C
- added C9: 47u, symbol CP
- added D3, D4: D, symbol D
- added IC8: LM741, symbol LM741
- added P12: 10k, symbol POT
- added R28, R29: 5k6, symbol R
- added R30: 4k7, symbol R
- added R31, R35: 1k, symbol R
- added R32, R34: 47, symbol R
- added R33: 6k8, symbol R
- added R36: 10k, symbol R
- added R37: 330k, symbol R
- added T4, T5: 2N3904, TO_SOT_Packages_THT:TO-92_Molded_Narrow, symbol 2N3904
Connections:
- new net: R32.1, T4.1 (E)
- new net: R30.1, R31.1, T4.2 (B)
- new net: C13.2, R28.2, T4.3 (C)
- new net: R34.1, T5.1 (E)
- new net: R35.1, R36.1, T5.2 (B)
- new net: C13.1, C8.2, R29.2, T5.3 (C)
- new net: R32.2, R33.1, R34.2
- new net: P12.1, P12.2, R30.2
- new net: D4.2 (A), R36.2
- new net: D3.1 (K), P12.3
- new net: C9.2, D3.2 (A), D4.1 (K)
- new net: C8.1, IC8.3 (+), R37.1
- new net +15V: IC8.7 (V+), R28.1, R29.1
- new net -15V: IC8.4 (V-), R33.2
- new net GND: R31.2, R35.2, R37.2
- new net ramp: C9.1
- new net triang: IC8.2 (-), IC8.6
- no-connect marks 0 -> 2
