File: sawtooh_osc.sch (KiCad schematic (older format))
At the start: 15 parts, among them IC1 4011, P10 4k7, P9 2k2, T1 2N3904, T2 Q_NJFET_DGS, T3 Q_NJFET_DGS

Commit message: falta sumador final
Connections:
- net ramp renamed sawtooh
Changed lines of the file:
@@
 $Descr A4 11693 8268
 encoding utf-8
-Sheet 2 4
+Sheet 2 7
 Title "Voltage Controlled Oscillator"
 Date ""
@@
 5V
 Text HLabel 7400 4400 2    60   Output ~ 0
-ramp
+sawtooh
 Text HLabel 4600 2800 1    60   Input ~ 0
 +15V
